Commit message: changes on urdf files and adding the ros2_control

File: description/clydedale_robot_core.urdf.xacro (robot description, xacro)
@@ -17,6 +17,17 @@
         <color rgba="0.5 0.5 0 1"/>
     </material>
+    <material name="red">
+        <color rgba="1 0 0 1"/>
+    </material>
     <!-- base_link -->
     <link name="base_link">
+    </link>
+     <!-- BASE_FOOTPRINT LINK -->
+    <joint name="base_footprint_joint" type="fixed">
+        <parent link="base_link"/>
+        <child link="base_footprint"/>
+        <origin xyz="0 0 0" rpy="0 0 0"/>
+    </joint>
+    <link name="base_footprint">
     </link>
     <!-- chassis -->
@@ -32,5 +43,5 @@
             </geometry>
             <material name="black"/>
-            <origin xyz="0.10 0 0.075" rpy="0 0 0"/>
+            <origin xyz="0.20 0 0.075" rpy="0 0 0"/>
         </visual>
         <collision>
@@ -38,8 +49,8 @@
                 <box size="0.4 0.3 0.15"/>
             </geometry>
-            <origin xyz="0.10 0 0.075" rpy="0 0 0"/>
+            <origin xyz="0.20 0 0.075" rpy="0 0 0"/>
         </collision>
         <xacro:inertial_box mass="0.5" x="0.4" y="0.3" z="0.15">
-            <origin xyz="0.10 0 0.075" rpy="0 0 0"/>
+            <origin xyz="0.20 0 0.075" rpy="0 0 0"/>
         </xacro:inertial_box>
     </link>
@@ -58,5 +69,5 @@
             <collision>
                 <geometry>
-                    <cylinder radius="0.05" length="0.04" />
+                    <sphere radius="0.05" length="0.04" />
                 </geometry>
                 <origin xyz="0 0 0" rpy="0 0 0" />
@@ -74,5 +85,5 @@
         <parent link="base_link" />
         <child link="left_wheel_front_link" />
-        <origin xyz="0.1 0.175 0" rpy="${pi/2} 0 0" />
+        <origin xyz="0.2 0.175 0" rpy="-${pi/2} 0 0" />
         <axis xyz="0 0 1" />
     </joint>
@@ -82,5 +93,5 @@
         <parent link="base_link" />
         <child link="left_wheel_back_link" />
-        <origin xyz="-0.1 0.175 0" rpy="${pi/2} 0 0" />
+        <origin xyz="0 0.175 0" rpy="-${pi/2} 0 0" />
         <axis xyz="0 0 1" />
     </joint>
@@ -90,5 +101,5 @@
         <parent link="base_link" />
         <child link="right_wheel_front_link" />
-        <origin xyz="0.1 -0.175 0" rpy="${pi/2} 0 0" />
+        <origin xyz="0.2 -0.175 0" rpy="${pi/2} 0 0" />
         <axis xyz="0 0 -1" />
     </joint>
@@ -98,5 +109,5 @@
         <parent link="base_link" />
         <child link="right_wheel_back_link" />
-        <origin xyz="-0.1 -0.175 0" rpy="${pi/2} 0 0" />
+        <origin xyz="0 -0.175 0" rpy="${pi/2} 0 0" />
         <axis xyz="0 0 -1" />
     </joint>

File: description/clydesdale_robot.urdf.xacro (robot description, xacro)
@@ -2,4 +2,6 @@
 <robot xmlns:xacro="http://www.ros.org/wiki/xacro"  name="clydesdale_robot">
     <xacro:include filename="clydedale_robot_core.urdf.xacro" />
-    <xacro:include filename="gazebo_control.urdf.xacro" />
+    <!-- <xacro:include filename="gazebo_control.urdf.xacro" /> -->
+    <xacro:include filename="lidar.xacro" />
+    <xacro:include filename="ros2_control.xacro"/>
 </robot>

File: description/gazebo_control.urdf.xacro (robot description, xacro)
@@ -4,8 +4,8 @@
         <plugin name="diff_drive" filename="libgazebo_ros_diff_drive.so">
             <!-- Wheel Information -->
-            <num_wheel_pairs>2</num_wheel_pairs>
-            <left_joint>left_wheel_front_joint</left_joint>
+            <!-- <num_wheel_pairs>2</num_wheel_pairs> -->
+            <!-- <left_joint>left_wheel_front_joint</left_joint> -->
             <left_joint>left_wheel_back_joint</left_joint>
-            <right_joint>right_wheel_front_joint</right_joint>
+            <!-- <right_joint>right_wheel_front_joint</right_joint> -->
             <right_joint>right_wheel_back_joint</right_joint>
             <wheel_separation>0.35</wheel_separation>

Commit message: adding joysticks

File: description/clydedale_robot_core.urdf.xacro (robot description, xacro)
@@ -88,5 +88,25 @@
         <axis xyz="0 0 1" />
     </joint>
-    <xacro:wheel_link prefix="left" place="front" />
+    <!-- <xacro:wheel_link prefix="left" place="front" /> -->
+    <link name="left_wheel_front_link">
+        <visual>
+            <geometry>
+                <cylinder radius="0.05" length="0.04" />
+            </geometry>
+            <material name="yellow" />
+        </visual>
+        <collision>
+            <geometry>
+                <sphere radius="0.05" length="0.04" />
+            </geometry>
+            <origin xyz="0 0 0" rpy="0 0 0" />
+        </collision>
+        <xacro:inertial_cylinder mass="0.1" length="0.04" radius="0.05">
+            <origin xyz="0 0 0" rpy="0 0 0" />
+        </xacro:inertial_cylinder>
+    </link>
+    <gazebo reference="left_wheel_front_link">
+        <material>Gazebo/Yellow</material>
+    </gazebo>
     <!--Left Wheel back-->
     <joint name="left_wheel_back_joint" type="continuous">

File: description/gazebo_control.urdf.xacro (robot description, xacro)
@@ -4,8 +4,8 @@
         <plugin name="diff_drive" filename="libgazebo_ros_diff_drive.so">
             <!-- Wheel Information -->
-            <!-- <num_wheel_pairs>2</num_wheel_pairs> -->
-            <!-- <left_joint>left_wheel_front_joint</left_joint> -->
+            <num_wheel_pairs>2</num_wheel_pairs>
+            <left_joint>left_wheel_front_joint</left_joint>
             <left_joint>left_wheel_back_joint</left_joint>
-            <!-- <right_joint>right_wheel_front_joint</right_joint> -->
+            <right_joint>right_wheel_front_joint</right_joint>
             <right_joint>right_wheel_back_joint</right_joint>
             <wheel_separation>0.35</wheel_separation>

Commit message: fixed error of tf

File: description/clydedale_robot_core.urdf.xacro (robot description, xacro)
@@ -20,4 +20,15 @@
         <color rgba="1 0 0 1"/>
     </material>
+     <!-- Constants for robot dimensions -->
+    <xacro:property name="chassis_mass" value="1.0"/>
+    <xacro:property name="chassis_length" value="0.3"/>
+    <xacro:property name="chassis_width" value="0.2"/>
+    <xacro:property name="chassis_height" value="0.15"/>
+    <xacro:property name="wheel_radius" value="0.033"/>
+    <xacro:property name="wheel_thickness" value="0.026"/>
+    <xacro:property name="wheel_mass" value="0.05"/>
+    <xacro:property name="wheel_offset_x" value="0.075"/>
+    <xacro:property name="wheel_offset_y" value="0.1285"/>
+    <xacro:property name="wheel_offset_z" value="0.015"/>
     <!-- base_link -->
     <link name="base_link">
@@ -35,22 +46,22 @@
         <parent link="base_link"/>
         <child link="chassis_link"/>
-        <origin xyz="-0.1 0 0"/>
+        <origin xyz="${-wheel_offset_x} 0 ${-wheel_offset_z}"/>
     </joint>
     <link name="chassis_link">
         <visual>
+            <origin xyz="${chassis_length/2} 0 ${chassis_height/2}"/>
             <geometry>
-                <box size="0.4 0.3 0.15"/>
+                <box size="${chassis_length} ${chassis_width} ${chassis_height}"/>
             </geometry>
             <material name="black"/>
-            <origin xyz="0.20 0 0.075" rpy="0 0 0"/>
         </visual>
         <collision>
+            <origin xyz="${chassis_length/2} 0 ${chassis_height/2}"/>
             <geometry>
-                <box size="0.4 0.3 0.15"/>
+                <box size="${chassis_length} ${chassis_width} ${chassis_height}"/>
             </geometry>
-            <origin xyz="0.20 0 0.075" rpy="0 0 0"/>
         </collision>
-        <xacro:inertial_box mass="0.5" x="0.4" y="0.3" z="0.15">
-            <origin xyz="0.20 0 0.075" rpy="0 0 0"/>
+        <xacro:inertial_box mass="0.5" x="${chassis_length}" y="${chassis_width}" z="${chassis_height}">
+            <origin xyz="${chassis_length/2} 0 ${chassis_height/2}" rpy="0 0 0"/>
         </xacro:inertial_box>
     </link>
@@ -63,16 +74,15 @@
             <visual>
                 <geometry>
-                    <cylinder radius="0.05" length="0.04" />
+                    <cylinder radius="${wheel_radius}" length="${wheel_thickness}"/>
                 </geometry>
-                <material name="yellow" />
+                <material name="blue"/>
             </visual>
             <collision>
                 <geometry>
-                    <sphere radius="0.05" length="0.04" />
+                    <sphere radius="${wheel_radius}"/>
                 </geometry>
-                <origin xyz="0 0 0" rpy="0 0 0" />
             </collision>
-            <xacro:inertial_cylinder mass="0.1" length="0.04" radius="0.05">
-                <origin xyz="0 0 0" rpy="0 0 0" />
+            <xacro:inertial_cylinder mass="${wheel_mass}" length="${wheel_thickness}" radius="${wheel_radius}">
+                <origin xyz="0 0 0" rpy="0 0 0"/>
             </xacro:inertial_cylinder>
         </link>
@@ -82,30 +92,14 @@
     </xacro:macro>
     <!--Left Wheel Front-->
-   <joint name="left_wheel_front_joint" type="continuous">
+   <joint name="left_wheel_front_joint" type="fixed">
         <parent link="base_link" />
         <child link="left_wheel_front_link" />
-        <origin xyz="0.2 0.175 0" rpy="-${pi/2} 0 0" />
+        <origin xyz="0.15 ${wheel_offset_y} 0" rpy="-${pi/2} 0 0" />
         <axis xyz="0 0 1" />
     </joint>
-    <!-- <xacro:wheel_link prefix="left" place="front" /> -->
-    <link name="left_wheel_front_link">
-        <visual>
-            <geometry>
-                <cylinder radius="0.05" length="0.04" />
-            </geometry>
-            <material name="yellow" />
-        </visual>
-        <collision>
-            <geometry>
-                <sphere radius="0.05" length="0.04" />
-            </geometry>
-            <origin xyz="0 0 0" rpy="0 0 0" />
-        </collision>
-        <xacro:inertial_cylinder mass="0.1" length="0.04" radius="0.05">
-            <origin xyz="0 0 0" rpy="0 0 0" />
-        </xacro:inertial_cylinder>
-    </link>
+    <xacro:wheel_link prefix="left" place="front" />
     <gazebo reference="left_wheel_front_link">
-        <material>Gazebo/Yellow</material>
+            <mu1 value="0.001"/>
+            <mu2 value="0.001"/>
     </gazebo>
     <!--Left Wheel back-->
@@ -113,22 +107,26 @@
         <parent link="base_link" />
         <child link="left_wheel_back_link" />
-        <origin xyz="0 0.175 0" rpy="-${pi/2} 0 0" />
-        <axis xyz="0 0 1" />
+        <origin xyz="0 ${wheel_offset_y} 0" rpy="-${pi/2} 0 0" />
+        <axis xyz="0 0 1"/>
     </joint>
     <xacro:wheel_link prefix="left" place="back" />
     <!--Right Wheel Front-->
-    <joint name="right_wheel_front_joint" type="continuous">
+    <joint name="right_wheel_front_joint" type="fixed">
         <parent link="base_link" />
         <child link="right_wheel_front_link" />
-        <origin xyz="0.2 -0.175 0" rpy="${pi/2} 0 0" />
+        <origin xyz="0.15 ${-wheel_offset_y}  0" rpy="${pi/2} 0 0" />
         <axis xyz="0 0 -1" />
     </joint>
     <xacro:wheel_link prefix="right" place="front" />
+    <gazebo reference="right_wheel_front_link">
+            <mu1 value="0.001"/>
+            <mu2 value="0.001"/>
+    </gazebo>
      <!--right Wheel Back-->
     <joint name="right_wheel_back_joint" type="continuous">
         <parent link="base_link" />
         <child link="right_wheel_back_link" />
-        <origin xyz="0 -0.175 0" rpy="${pi/2} 0 0" />
-        <axis xyz="0 0 -1" />
+        <origin xyz="0 ${-wheel_offset_y} 0" rpy="${pi/2} 0 0" />
+        <axis xyz="0 0 -1"/>
     </joint>
     <xacro:wheel_link prefix="right" place="back" />

File: description/clydesdale_robot.urdf.xacro (robot description, xacro)
@@ -1,7 +1,12 @@
 <?xml version="1.0"?>
 <robot xmlns:xacro="http://www.ros.org/wiki/xacro"  name="clydesdale_robot">
+    <xacro:arg name="use_ros2_control" default="true"/>
     <xacro:include filename="clydedale_robot_core.urdf.xacro" />
-    <!-- <xacro:include filename="gazebo_control.urdf.xacro" /> -->
     <xacro:include filename="lidar.xacro" />
-    <xacro:include filename="ros2_control.xacro"/>
+    <xacro:if value="$(arg use_ros2_control)">
+        <xacro:include filename="ros2_control.xacro"/>
+    </xacro:if>
+    <xacro:unless value="$(arg use_ros2_control)">
+        <xacro:include filename="gazebo_control.urdf.xacro" />
+    </xacro:unless>
 </robot>

File: description/gazebo_control.urdf.xacro (robot description, xacro)
@@ -4,5 +4,9 @@
         <plugin name="diff_drive" filename="libgazebo_ros_diff_drive.so">
             <!-- Wheel Information -->
-            <num_wheel_pairs>2</num_wheel_pairs>
+            <left_joint>left_wheel_back_joint</left_joint>
+            <right_joint>right_wheel_back_joint</right_joint>
+            <wheel_separation>0.295</wheel_separation>
+            <wheel_diameter>0.066</wheel_diameter>
+            <!-- <num_wheel_pairs>2</num_wheel_pairs>
             <left_joint>left_wheel_front_joint</left_joint>
             <left_joint>left_wheel_back_joint</left_joint>
@@ -10,5 +14,5 @@
             <right_joint>right_wheel_back_joint</right_joint>
             <wheel_separation>0.35</wheel_separation>
-            <wheel_diameter>0.1</wheel_diameter>
+            <wheel_diameter>0.1</wheel_diameter> -->
             <!-- Limits -->
             <max_wheel_torque>200</max_wheel_torque>
